File: is31fl3730_grid.kicad_pcb (KiCad board)
At the start: 2 copper layers, 134 parts, among them J1 Conn_01x06, U1 IS31FL3730

Commit message: Fix matrix
Parts:
- removed the D106 at (126.7, 126.7)
- removed the D120 at (130.5, 126.7)
- removed the D22 at (103.8, 126.7)
- removed the D36 at (107.6, 126.7)
- removed the D50 at (111.4, 126.7)
- removed the D64 at (115.2, 126.7)
- removed the D78 at (119.0, 126.7)
- removed the D8 at (100.0, 126.7)
- removed the D92 at (122.9, 126.7)
- added D100: LED, LED_SMD:LED_0805_2012Metric, F.Cu at (158.4, 77.1)
- added D114: LED, LED_SMD:LED_0805_2012Metric, F.Cu at (166.0, 77.1)
- added D16: LED, LED_SMD:LED_0805_2012Metric, F.Cu at (112.7, 77.1)
- added D2: LED, LED_SMD:LED_0805_2012Metric, F.Cu at (105.1, 77.1)
- added D30: LED, LED_SMD:LED_0805_2012Metric, F.Cu at (120.3, 77.1)
- added D44: LED, LED_SMD:LED_0805_2012Metric, F.Cu at (127.9, 77.1)
- added D58: LED, LED_SMD:LED_0805_2012Metric, F.Cu at (135.6, 77.1)
- added D72: LED, LED_SMD:LED_0805_2012Metric, F.Cu at (143.2, 77.1)
- added D86: LED, LED_SMD:LED_0805_2012Metric, F.Cu at (150.8, 77.1)
- added R2: 10kR, Resistor_SMD:R_0805_2012Metric, B.Cu at (90.1, 88.4)
- added REF**: Logo_WM, Symbol:Logo_WM, F.Cu at (97.0, 97.9)
- C1, J1, U1: moved to B.Cu
- moved D124 66.3 mm to (169.8, 88.6), turned to 225 degrees
- moved D125 66.3 mm to (169.8, 92.4), turned to 225 degrees
- moved D126 66.3 mm to (169.8, 96.2), turned to 225 degrees
- moved D122 66.3 mm to (169.8, 81.0), turned to 225 degrees
- moved D123 66.3 mm to (169.8, 84.8), turned to 225 degrees
- moved D121 66.3 mm to (169.8, 77.1), turned to 225 degrees
- moved D110 64.1 mm to (162.2, 88.6), turned to 225 degrees
- moved D111 64.1 mm to (162.2, 92.4), turned to 225 degrees
- moved D112 64.1 mm to (162.2, 96.2), turned to 225 degrees
- moved D108 64.1 mm to (162.2, 81.0), turned to 225 degrees
- moved D109 64.1 mm to (162.2, 84.8), turned to 225 degrees
- moved D107 64.1 mm to (162.2, 77.1), turned to 225 degrees
- moved D96 62.1 mm to (154.6, 88.6), turned to 225 degrees
- moved D97 62.1 mm to (154.6, 92.4), turned to 225 degrees
- moved D98 62.1 mm to (154.6, 96.2), turned to 225 degrees
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- renumbered D100 to D106, D114 to D120, D16 to D22, D30 to D36, D44 to D50, D58 to D64, D72 to D78, D2 to D8, D86 to D92
Connections:
- D1 pad 1: R1 -> C1
- D1 pad 2: C1 -> R1
- D10 pad 1: C1 -> R3
- D10 pad 2: R5 -> C1
- D101 pad 1: R2 -> C8
- D101 pad 2: C8 -> R3
- D102 pad 2: R2 -> R4
- D103 pad 1: R3 -> C8
- D103 pad 2: C8 -> R5
- D104 pad 2: R3 -> R6
- D105 pad 1: R4 -> C8
- D105 pad 2: C8 -> R7
- D106 pad 1: C8 -> R1
- D106 pad 2: R1 -> C8
- D107 pad 1: R5 -> R2
- D108 pad 1: C8 -> R3
- D108 pad 2: R5 -> C8
- D109 pad 1: R6 -> R4
- D11 pad 1: R6 -> R4
- D110 pad 1: C8 -> R5
- D110 pad 2: R6 -> C8
- D111 pad 1: R7 -> R6
- D112 pad 1: C8 -> R7
- D112 pad 2: R7 -> C8
- D113 pad 1: R1 -> C9
- D113 pad 2: C9 -> R1
- D115 pad 1: R2 -> C9
- D115 pad 2: C9 -> R3
- D116 pad 2: R2 -> R4
- D117 pad 1: R3 -> C9
- D117 pad 2: C9 -> R5
- D118 pad 2: R3 -> R6
- D119 pad 1: R4 -> C9
- D119 pad 2: C9 -> R7
- D12 pad 1: C1 -> R5
- D12 pad 2: R6 -> C1
- D120 pad 1: C9 -> R1
- D120 pad 2: R1 -> C9
- D121 pad 1: R5 -> R2
- D122 pad 1: C9 -> R3
- D122 pad 2: R5 -> C9
- D123 pad 1: R6 -> R4
- D124 pad 1: C9 -> R5
- D124 pad 2: R6 -> C9
- D125 pad 1: R7 -> R6
- D126 pad 1: C9 -> R7
- D126 pad 2: R7 -> C9
- D13 pad 1: R7 -> R6
- D14 pad 1: C1 -> R7
- D14 pad 2: R7 -> C1
- D15 pad 1: R1 -> C2
- D15 pad 2: C2 -> R1
- D17 pad 1: R2 -> C2
- D17 pad 2: C2 -> R3
- D18 pad 2: R2 -> R4
- D19 pad 1: R3 -> C2
- D19 pad 2: C2 -> R5
- D20 pad 2: R3 -> R6
- D21 pad 1: R4 -> C2
- D21 pad 2: C2 -> R7
- D22 pad 1: C2 -> R1
- D22 pad 2: R1 -> C2
- D23 pad 1: R5 -> R2
- D24 pad 1: C2 -> R3
- D24 pad 2: R5 -> C2
- D25 pad 1: R6 -> R4
- D26 pad 1: C2 -> R5
- D26 pad 2: R6 -> C2
- D27 pad 1: R7 -> R6
- D28 pad 1: C2 -> R7
- D28 pad 2: R7 -> C2
- D29 pad 1: R1 -> C3
- D29 pad 2: C3 -> R1
- D3 pad 1: R2 -> C1
- D3 pad 2: C1 -> R3
- D31 pad 1: R2 -> C3
- D31 pad 2: C3 -> R3
- D32 pad 2: R2 -> R4
- D33 pad 1: R3 -> C3
- D33 pad 2: C3 -> R5
- D34 pad 2: R3 -> R6
- D35 pad 1: R4 -> C3
- D35 pad 2: C3 -> R7
- D36 pad 1: C3 -> R1
- D36 pad 2: R1 -> C3
- D37 pad 1: R5 -> R2
- D38 pad 1: C3 -> R3
- D38 pad 2: R5 -> C3
- D39 pad 1: R6 -> R4
- D4 pad 2: R2 -> R4
- D40 pad 1: C3 -> R5
- D40 pad 2: R6 -> C3
- D41 pad 1: R7 -> R6
- D42 pad 1: C3 -> R7
- D42 pad 2: R7 -> C3
- D43 pad 1: R1 -> C4
- D43 pad 2: C4 -> R1
- D45 pad 1: R2 -> C4
- D45 pad 2: C4 -> R3
- D46 pad 2: R2 -> R4
- D47 pad 1: R3 -> C4
- D47 pad 2: C4 -> R5
- D48 pad 2: R3 -> R6
- D49 pad 1: R4 -> C4
- D49 pad 2: C4 -> R7
- D5 pad 1: R3 -> C1
- D5 pad 2: C1 -> R5
- D50 pad 1: C4 -> R1
- D50 pad 2: R1 -> C4
- D51 pad 1: R5 -> R2
- D52 pad 1: C4 -> R3
- D52 pad 2: R5 -> C4
- D53 pad 1: R6 -> R4
- D54 pad 1: C4 -> R5
- D54 pad 2: R6 -> C4
- D55 pad 1: R7 -> R6
- D56 pad 1: C4 -> R7
- D56 pad 2: R7 -> C4
- D57 pad 1: R1 -> C5
- D57 pad 2: C5 -> R1
- D59 pad 1: R2 -> C5
- D59 pad 2: C5 -> R3
- D6 pad 2: R3 -> R6
- D60 pad 2: R2 -> R4
- D61 pad 1: R3 -> C5
- D61 pad 2: C5 -> R5
- D62 pad 2: R3 -> R6
- D63 pad 1: R4 -> C5
- D63 pad 2: C5 -> R7
- D64 pad 1: C5 -> R1
- D64 pad 2: R1 -> C5
- D65 pad 1: R5 -> R2
- D66 pad 1: C5 -> R3
- D66 pad 2: R5 -> C5
- D67 pad 1: R6 -> R4
- D68 pad 1: C5 -> R5
- D68 pad 2: R6 -> C5
- D69 pad 1: R7 -> R6
- D7 pad 1: R4 -> C1
- D7 pad 2: C1 -> R7
- D70 pad 1: C5 -> R7
- D70 pad 2: R7 -> C5
- D71 pad 1: R1 -> C6
- D71 pad 2: C6 -> R1
- D73 pad 1: R2 -> C6
- D73 pad 2: C6 -> R3
- D74 pad 2: R2 -> R4
- D75 pad 1: R3 -> C6
- D75 pad 2: C6 -> R5
- D76 pad 2: R3 -> R6
- D77 pad 1: R4 -> C6
- D77 pad 2: C6 -> R7
- D78 pad 1: C6 -> R1
- D78 pad 2: R1 -> C6
- D79 pad 1: R5 -> R2
- D8 pad 1: C1 -> R1
- D8 pad 2: R1 -> C1
- D80 pad 1: C6 -> R3
- D80 pad 2: R5 -> C6
- D81 pad 1: R6 -> R4
- D82 pad 1: C6 -> R5
- D82 pad 2: R6 -> C6
- D83 pad 1: R7 -> R6
- D84 pad 1: C6 -> R7
- D84 pad 2: R7 -> C6
- D85 pad 1: R1 -> C7
- D85 pad 2: C7 -> R1
- D87 pad 1: R2 -> C7
- D87 pad 2: C7 -> R3
- D88 pad 2: R2 -> R4
- D89 pad 1: R3 -> C7
- D89 pad 2: C7 -> R5
- D9 pad 1: R5 -> R2
- D90 pad 2: R3 -> R6
- D91 pad 1: R4 -> C7
- D91 pad 2: C7 -> R7
- D92 pad 1: C7 -> R1
- D92 pad 2: R1 -> C7
- D93 pad 1: R5 -> R2
- D94 pad 1: C7 -> R3
- D94 pad 2: R5 -> C7
- D95 pad 1: R6 -> R4
- D96 pad 1: C7 -> R5
- D96 pad 2: R6 -> C7
- D97 pad 1: R7 -> R6
- D98 pad 1: C7 -> R7
- D98 pad 2: R7 -> C7
- D99 pad 1: R1 -> C8
- D99 pad 2: C8 -> R1
Routing:
- net C9: track 0.00 -> 133.7 mm, vias 0 -> 7
- net C8: track 0.00 -> 125.5 mm, vias 0 -> 7
- net C7: track 0.00 -> 117.0 mm, vias 0 -> 7
- net C6: track 0.00 -> 108.6 mm, vias 0 -> 7
- net C5: track 0.00 -> 101.1 mm, vias 0 -> 7
- net C4: track 0.00 -> 96.7 mm, vias 0 -> 7
- net C3: track 0.00 -> 90.9 mm, vias 0 -> 8
- net R7: track 0.00 -> 87.2 mm, vias 0 -> 1
- net R1: track 0.00 -> 87.0 mm, vias 0 -> 1
- net R2: track 0.00 -> 86.5 mm, vias 0 -> 1
- net R6: track 0.00 -> 85.4 mm, vias 0 -> 1
- net R5: track 0.00 -> 84.2 mm, vias 0 -> 1
- net C2: track 0.00 -> 84.2 mm, vias 0 -> 8
- net R4: track 0.00 -> 83.9 mm, vias 0 -> 1
- net R3: track 0.00 -> 82.5 mm, vias 0 -> 1
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- added copper zone on B.Cu, net GND
- added copper zone on F.Cu, net GND
Other:
- board outline added: 87 x 31.1 mm
- board text added: "AUD"
- board text added: "C0"
- board text added: "C2"
- board text added: "C4"
- board text added: "C6"
- board text added: "GND"
- board text added: "SCL"
- board text added: "SDA"
- board text added: "SDB"
- board text added: "VCC"
- board text added: "v0.0.0 05/17/20"
